File: elec/layout/default/demo.kicad_pcb (KiCad board)
At the start: 4 copper layers, 29.9 x 31.9 mm, 32 parts, among them U1 ?, U2 ?, U3 ?, U4 ?, U5 KMR211NGLFS (Tactile Switches), U6 ?, U7 ?

Commit message: [ROUTE] fix
Other:
- board size 29.9 x 31.9 mm -> 30 x 31.9 mm
Changed lines of the file:
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@@
 			(at 0 0 0)
 			(layer "F.SilkS")
+			(hide yes)
 			(effects
 				(font
@@
 			(at 0 0 90)
 			(layer "F.SilkS")
+			(hide yes)
 			(effects
 				(font
@@
 			(unlocked yes)
 			(layer "F.SilkS")
+			(hide yes)
 			(effects
 				(font
@@
 		)
 		(fp_text user "*"
-			(at -1.4478 -2.6921 0)
-			(unlocked yes)
-			(layer "F.SilkS")
-			(effects
-				(font
-					(size 1 1)
-					(thickness 0.15)
-				)
-			)
-		)
-		(fp_text user "*"
-			(at -1.4478 -2.6921 0)
+			(at -1.7994 -1.6446 0)
 			(layer "F.SilkS")
 			(effects
@@
 			(at -2 0 180)
 			(layer "F.SilkS")
+			(hide yes)
 			(effects
 				(font
@@
 			(at 0 0.0082 90)
 			(layer "F.SilkS")
+			(hide yes)
 			(effects
 				(font
@@
 			(at 0 -1.17 0)
 			(layer "F.SilkS")
+			(hide yes)
 			(effects
 				(font
@@
 			(at -2 0 0)
 			(layer "F.SilkS")
+			(hide yes)
 			(effects
 				(font
@@
 			(at 0 -1.17 0)
 			(layer "F.SilkS")
+			(hide yes)
 			(effects
 				(font
@@
 	(gr_rect
 		(start 125.1 87.6)
-		(end 155 119.5)
+		(end 155.1 119.5)
 		(stroke
 			(width 0.1)

Commit message: [PCB] remove release
Parts:
- C7, C8: value 50V 20pF C0G ±5% 0402 Multilayer Ceramic Capacitors MLCC - SMD/SMT ROHS -> 50V 22pF C0G ±5% 0402 Multilayer Ceramic Capacitors MLCC - SMD/SMT ROHS
- moved C3 26.8 mm to (152.7, 116.4), turned to 0 degrees
- moved C4 24.8 mm to (152.7, 115.4), turned to 0 degrees
- moved C5 22.9 mm to (152.7, 114.3), turned to 0 degrees
- moved U3 22.2 mm to (147.8, 114.8), turned to 90 degrees
- moved C1 21.9 mm to (152.7, 94.6)
- moved C2 21.9 mm to (150.2, 94.6)
- moved U2 21.9 mm to (151.4, 92.0)
- moved C6 21.1 mm to (152.7, 113.3), turned to 0 degrees
- moved R4 2.20 mm to (130.7, 103.4)
- moved R5 2.20 mm to (133.8, 114.2)
- moved R6 2.20 mm to (137.7, 102.4)
- moved R7 2.20 mm to (137.7, 103.4)
- moved U7 2.20 mm to (134.1, 99.4)
- moved C13 2.20 mm to (139.5, 109.3)
- moved C7 2.20 mm to (130.0, 116.5)
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Other:
- board size 30 x 31.9 mm -> 29.3 x 31.9 mm

Commit message: [DEMO] remove prompts
Parts:
- moved R1 0.81 mm to (144.1, 105.1)
- moved R2 0.81 mm to (144.0, 101.3)
- moved U1 0.81 mm to (149.1, 102.2)
- moved C1 0.63 mm to (152.1, 94.6)
- moved C16 0.63 mm to (138.8, 104.5)
- moved C2 0.63 mm to (149.6, 94.6)
- moved R3 0.63 mm to (128.1, 109.3)
- moved R4 0.63 mm to (130.1, 103.4)
- moved R5 0.63 mm to (133.2, 114.2)
- moved R6 0.63 mm to (137.1, 102.4)
- moved R7 0.63 mm to (137.1, 103.4)
- moved U5 0.63 mm to (133.3, 91.9)
- moved U7 0.63 mm to (133.4, 99.4)
- moved C10 0.63 mm to (138.8, 105.5)
- moved C12 0.63 mm to (128.1, 105.5)
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Routing:
- added copper zone on In1.Cu, net power_supply-vcc
- added copper zone on B.Cu, net usb_connector-gnd-1
- added copper zone on F.Cu, net usb_connector-gnd-1
- added copper zone on In2.Cu, net usb_connector-gnd-1
- removed copper zone on B.Cu, net usb_connector-vcc
